Commit message: schunk_description: sets urdf joints as the robot specification

File: schunk_description/urdf/lwa4p/lwa4p.urdf.xacro (robot description, xacro)
@@ -50,5 +50,5 @@
       <child link="${name}_1_link"/>
       <axis xyz="0 0 1"/>
-      <limit effort="370" velocity="2.0" lower="${-6.28 + safety_offset}" upper="${6.28 - safety_offset}"/>
+      <limit effort="370" velocity="2.0" lower="${-2.97 + safety_offset}" upper="${2.97 - safety_offset}"/>
       <!--safety_controller k_position="20" k_velocity="50" soft_lower_limit="${-6.28 + 0.01}" soft_upper_limit="${6.28 - 0.01}" /-->
     </joint>
@@ -82,5 +82,5 @@
       <child link="${name}_2_link"/>
       <axis xyz="0 0 1"/>
-      <limit effort="370" velocity="2.0" lower="${-2.09 + safety_offset}" upper="${2.09 - safety_offset}"/>
+      <limit effort="370" velocity="2.0" lower="${-2.97 + safety_offset}" upper="${2.97 - safety_offset}"/>
       <!--safety_controller k_position="20" k_velocity="50" soft_lower_limit="${-2.09 + 0.01}" soft_upper_limit="${2.09 - 0.01}" /-->
     </joint>
@@ -146,5 +146,5 @@
       <child link="${name}_4_link"/>
       <axis xyz="0 0 1" />
-      <limit effort="176" velocity="2.0" lower="${-2.09 + safety_offset}" upper="${2.09 - safety_offset}"/>
+      <limit effort="176" velocity="2.0" lower="${-2.97 + safety_offset}" upper="${2.97 - safety_offset}"/>
       <!--safety_controller k_position="20" k_velocity="25" soft_lower_limit="${-2.09 + 0.01}" soft_upper_limit="${2.09 - 0.01}" /-->
     </joint>
@@ -178,5 +178,5 @@
       <child link="${name}_5_link"/>
       <axis xyz="0 0 1" />
-      <limit effort="41.6" velocity="2.0" lower="${-6.28 + safety_offset}" upper="${6.28 - safety_offset}" />
+      <limit effort="41.6" velocity="2.0" lower="${-2.97 + safety_offset}" upper="${2.97 - safety_offset}" />
       <!--safety_controller k_position="20" k_velocity="25" soft_lower_limit="${-6.28 + 0.01}" soft_upper_limit="${6.28 - 0.01}" /-->
     </joint>
@@ -210,5 +210,5 @@
       <child link="${name}_6_link"/>
       <axis xyz="0 0 1" />
-      <limit effort="20.1" velocity="2.0" lower="${-2.09 + safety_offset}" upper="${2.09 - safety_offset}" />
+      <limit effort="20.1" velocity="2.0" lower="${-2.97 + safety_offset}" upper="${2.97 - safety_offset}" />
       <!--safety_controller k_position="20" k_velocity="25" soft_lower_limit="${-2.09 + 0.01}" soft_upper_limit="${2.09 - 0.01}" /-->
     </joint>
