Commit message: schunk_description: changed linear limit for angular limit. Visualization needs to be fixed

File: schunk_description/urdf/pg70/pg70.urdf.xacro (robot description, xacro)
@@ -31,5 +31,6 @@
       <child link="${name}_finger_left_link" />
       <axis xyz="0 1 0" />
-      <limit effort="10" lower="-0.001" upper="0.061" velocity="2.0"/>
+      <!--limit effort="10" lower="-0.001" upper="0.061" velocity="2.0"/-->
+      <limit effort="10" lower="-0.001" upper="1.15" velocity="2.0"/>
     </joint>
     <link name="${name}_finger_left_link">
